File: keypadprototype.kicad_pcb (KiCad board)
At the start: 2 copper layers, 28 parts, among them SW1 SW_Push, U1 ATmega32U4-A, Y1 16MHz

Commit message: PCB Prototype - No Wiring 8/5
Parts:
- moved C4 74.5 mm to (85.8, 129.5), turned to 135 degrees
- moved USB1 73.3 mm to (91.3, 55.0), turned to -90 degrees
- moved C3 73.1 mm to (99.1, 135.1), turned to 45 degrees
- moved R3 63.2 mm to (92.9, 63.5), turned to 90 degrees
- moved C1 63.2 mm to (100.8, 118.3), turned to 45 degrees
- moved R2 62.9 mm to (90.5, 63.5), turned to 90 degrees
- moved C2 60.8 mm to (95.2, 113.5), turned to 135 degrees
- moved C5 60.3 mm to (104.4, 129.3), turned to -135 degrees
- moved U1 58.7 mm to (95.2, 125.4), turned to -135 degrees
- moved C6 58.2 mm to (85.1, 120.0), turned to -45 degrees
- moved R1 55.8 mm to (92.9, 135.7), turned to 135 degrees
- moved Y1 55.4 mm to (87.3, 117.5), turned to 45 degrees
- moved C7 53.1 mm to (89.8, 115.2), turned to 135 degrees
- moved R4 39.9 mm to (97.6, 111.1), turned to 135 degrees
- moved F1 36.9 mm to (106.4, 111.9), turned to -135 degrees
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Other:
- board outline added: 82.5 x 101.6 mm

Commit message: wiring 8/7
Parts:
- moved R1 13.1 mm to (87.2, 147.5)
- moved C3 13.1 mm to (93.4, 146.8)
- moved C4 13.1 mm to (80.1, 141.3)
- moved C5 13.1 mm to (98.7, 141.0)
- moved U1 10.6 mm to (90.5, 134.9)
- moved Y1 10.3 mm to (78.6, 123.0)
- moved C6 10.3 mm to (76.3, 125.5)
- moved C7 9.30 mm to (81.8, 119.9)
- moved C1 8.59 mm to (96.0, 125.4)
- moved F1 8.59 mm to (101.6, 119.1)
- moved SW1 8.59 mm to (106.8, 128.7)
- moved C2 6.80 mm to (91.1, 118.9)
- moved R4 6.80 mm to (93.5, 116.5)
- moved R2 1.47 mm to (90.5, 65.0)
- moved R3 1.47 mm to (92.9, 65.0)
Routing:
- net GND: track 0.00 -> 32.6 mm
- net Net-(U1-XTAL2): track 0.00 -> 17.4 mm
- net Net-(U1-XTAL1): track 0.00 -> 13.1 mm
- net Net-(D3-A): track 0.00 -> 7.84 mm
- net Net-(D2-A): track 0.00 -> 7.84 mm
- net Net-(D1-A): track 0.00 -> 7.84 mm
- net Net-(D6-A): track 0.00 -> 7.84 mm
- net Net-(D5-A): track 0.00 -> 7.84 mm
- net Net-(D4-A): track 0.00 -> 7.84 mm
- net +5V: track 0.00 -> 7.64 mm
